Commit message: fix xacro(not complete)

File: simulation/urdf/wheel.urdf.xacro (robot description, xacro)
@@ -2,15 +2,16 @@
 <robot name="wheel" xmlns:xacro="http://www.ros.org/wiki/xacro">
   <!-- Wheels -->
-  <property name="wheel_radius" value="0.2" />
-  <property name="wheel_height" value="0.1" />
-  <property name="wheel_mass" value="1.5" /> <!-- in kg-->
-  <property name="base_x_origin_to_wheel_origin" value="0.25" />
-  <property name="base_y_origin_to_wheel_origin" value="0.3" />
-  <property name="base_z_origin_to_wheel_origin" value="0.0" />
-  <macro name="cylinder_inertia" params="m r h">
+  <xacro:property name="wheel_radius" value="0.2" />
+  <xacro:property name="wheel_height" value="0.1" />
+  <xacro:property name="wheel_mass" value="1.5" /> <!-- in kg-->
+  <xacro:property name="base_x_origin_to_wheel_origin" value="0.25" />
+  <xacro:property name="base_y_origin_to_wheel_origin" value="0.3" />
+  <xacro:property name="base_z_origin_to_wheel_origin" value="0.0" />
+  <xacro:property name="M_PI" value="3.1415926535897931" />
+  <xacro:macro name="cylinder_inertia" params="m r h">
     <inertia  ixx="${m*(3*r*r+h*h)/12}" ixy = "0" ixz = "0"
               iyy="${m*(3*r*r+h*h)/12}" iyz = "0"
               izz="${m*r*r/2}" />
-  </macro>
+  </xacro:macro>
   <xacro:macro name="wheel" params="fb lr parent translateX translateY flipY"> <!--fb : front, back ; lr: left, right -->
     <link name="${fb}_${lr}_wheel">
@@ -31,5 +32,5 @@
         <mass value="${wheel_mass}" />
         <origin xyz="0 0 0" />
-        <cylinder_inertia  m="${wheel_mass}" r="${wheel_radius}" h="${wheel_height}" />
+        <xacro:cylinder_inertia  m="${wheel_mass}" r="${wheel_radius}" h="${wheel_height}" />
       </inertial>
     </link>
@@ -43,4 +44,5 @@
       <turnGravityOff>false</turnGravityOff>
     </gazebo>
+    <!-- <ros2_control name="SkidSteerDriveController" type="system"> -->
     <joint name="${fb}_${lr}_wheel_joint" type="continuous">
       <parent link="${parent}"/>
@@ -62,4 +64,5 @@
       </actuator>
     </transmission>
+    <!-- </ros2_control> -->
   </xacro:macro>
 </robot>

File: simulation/urdf/wheel_robot_base.urdf.xacro (robot description, xacro)
@@ -2,25 +2,27 @@
 <robot name="wheel_robot_base" xmlns:xacro="http://www.ros.org/wiki/xacro">
   <!-- Included URDF/XACRO Files -->
-  <xacro:include filename="$(find model_pkg)/urdf/materials.urdf.xacro" />
-  <xacro:include filename="$(find model_pkg)/urdf/wheel.urdf.xacro" />
+  <xacro:include filename="$(find journal1-sim)/urdf/materials.urdf.xacro" />
+  <xacro:include filename="$(find journal1-sim)/urdf/wheel.urdf.xacro" />
   <!-- PROPERTY LIST -->
   <!--All units in m-kg-s-radians unit system -->
   <property name="M_PI" value="3.1415926535897931" />
   <!-- Main Body-base -->
-  <property name="base_x_size" value="1.0" />
-  <property name="base_y_size" value="0.5" />
-  <property name="base_z_size" value="0.25" />
-  <property name="base_mass" value="70" /> <!-- in kg-->
+  <xacro:property name="base_x_size" value="1.0" />
+  <xacro:property name="base_y_size" value="0.5" />
+  <xacro:property name="base_z_size" value="0.25" />
+  <xacro:property name="base_mass" value="70" /> <!-- in kg-->
+  <xacro:property name="wheel_radius" value="0.2" />
+  <xacro:property name="base_z_origin_to_wheel_origin" value="0.0" />
   <!--Inertial macros for the box and cylinder. Units are kg*m^2-->
-  <macro name="box_inertia" params="m x y z">
+  <xacro:macro name="box_inertia" params="m x y z">
     <inertia  ixx="${m*(y*y+z*z)/12}" ixy = "0" ixz = "0"
               iyy="${m*(x*x+z*z)/12}" iyz = "0"
               izz="${m*(x*x+z*z)/12}" />
-  </macro>
+  </xacro:macro>
   <!-- dummy link -->
   <!-- <link name="odom" /> -->
   <!-- BASE-FOOTPRINT -->
   <!-- base_link is a fictitious link(frame) that is on the ground right below base_body_link origin -->
-  <link name="base_foot_link">
+  <link name="base_link">
     <inertial>
       <mass value="0.0001" />
@@ -42,11 +44,11 @@
     <child link="odom" />
   </joint> -->
-  <gazebo reference="base_body_link">
+  <gazebo reference="base_link">
     <turnGravityOff>false</turnGravityOff>
   </gazebo>
-  <joint name="wheel_joint" type="fixed">
+  <joint name="base_link_joint" type="fixed">
     <origin xyz="0 0 ${wheel_radius - base_z_origin_to_wheel_origin}" rpy="0 0 0" />
-    <parent link="base_body_link"/>
-    <child link="base_foot_link" />
+    <parent link="base_link"/>
+    <child link="base_body_link" />
   </joint>
   <!-- BASE-LINK -->
@@ -57,5 +59,5 @@
       <origin xyz="0 0 0" />
       <!--The 3x3 rotational inertia matrix. -->
-      <box_inertia  m="${base_mass}" x="${base_x_size}" y="${base_y_size}" z="${base_z_size}"/>
+      <xacro:box_inertia  m="${base_mass}" x="${base_x_size}" y="${base_y_size}" z="${base_z_size}"/>
     </inertial>
     <visual>
@@ -78,10 +80,10 @@
   </gazebo>
   <!-- WHEELs -->
-  <wheel fb="front" lr="right" parent="base_foot_link" translateX="1" translateY="-1" flipY="-1"/>
-  <wheel fb="front" lr="left" parent="base_foot_link" translateX="1" translateY="1" flipY="-1"/>
-  <wheel fb="back" lr="right" parent="base_foot_link" translateX="-1" translateY="-1" flipY="-1"/>
-  <wheel fb="back" lr="left" parent="base_foot_link" translateX="-1" translateY="1" flipY="-1"/>
+  <xacro:wheel fb="front" lr="right" parent="base_body_link" translateX="1" translateY="-1" flipY="-1"/>
+  <xacro:wheel fb="front" lr="left" parent="base_body_link" translateX="1" translateY="1" flipY="-1"/>
+  <xacro:wheel fb="back" lr="right" parent="base_body_link" translateX="-1" translateY="-1" flipY="-1"/>
+  <xacro:wheel fb="back" lr="left" parent="base_body_link" translateX="-1" translateY="1" flipY="-1"/>
   <gazebo>
-    <plugin name="skid_steer_drive_controller" filename="libgazebo_ros_skid_steer_drive.so">
+    <plugin name="skid_steer_drive_controller" filename="libgazebo_ros_steer_drive.so">
       <alwaysOn>true</alwaysOn>
       <updateRate>50.0</updateRate>
@@ -94,17 +96,21 @@
       <torque>35</torque>
       <broadcastTF>1</broadcastTF>
-      <odometryFrame>odom</odometryFrame>
+      <odometryFrame>map</odometryFrame>
       <odometryTopic>odom</odometryTopic>
       <commandTopic>cmd_vel</commandTopic>
-      <robotBaseFrame>base_body_link</robotBaseFrame>
+      <robotBaseFrame>base_link</robotBaseFrame>
     </plugin>
-    <plugin name="gazebo_ros_control" filename="libgazebo_ros_control.so" >
-    </plugin>
+    <!-- <plugin name="gazebo_ros2_control" filename="libgazebo_ros2_control.so" >
+    </plugin> -->
   </gazebo>
   <xacro:arg name="gpu" default="true"/>
   <xacro:property name="gpu" value="$(arg gpu)" />
-  <xacro:include filename="$(find model_pkg)/urdf/VLP-16.urdf.xacro"/>
+  <!-- <xacro:include filename="$(find journal1-sim)/urdf/VLP-16.urdf.xacro"/>
   <VLP-16 parent="base_body_link" name="velodyne" topic="/points_raw" hz="10" samples="440" gpu="${gpu}">
     <origin xyz="0 0 0.4" rpy="0 0 0" />
-  </VLP-16>
+  </VLP-16> -->
+  <xacro:include filename="$(find velodyne_description)/urdf/VLP-16.urdf.xacro"/>
+  <xacro:VLP-16 parent="base_link" name="velodyne" topic="/points_raw" organize_cloud="false" hz="10" samples="440" gpu="${gpu}">
+    <origin xyz="0 0 0.4" rpy="0 0 0" />
+  </xacro:VLP-16>
 </robot>

Commit message: fix comment for autoware

File: simulation/urdf/wheel.urdf.xacro (robot description, xacro)
@@ -14,5 +14,5 @@
               izz="${m*r*r/2}" />
   </xacro:macro>
-  <xacro:macro name="wheel" params="fb lr parent translateX translateY flipY"> <!--fb : front, back ; lr: left, right -->
+  <xacro:macro name="wheel" params="fb lr parent translateX translateY flipY"> <!--fb , front, back ; lr, left, right -->
     <link name="${fb}_${lr}_wheel">
       <visual>
