Commit message: fix xacro

File: simulation/urdf/smagv/smagv.urdf.xacro (robot description, xacro)
@@ -254,5 +254,4 @@
     <xacro:include filename="$(find velodyne_description)/urdf/VLP-16.urdf.xacro"/>
     <xacro:VLP-16 parent="base_link" name="velodyne" topic="/sensing/lidar/concatenated/pointcloud" hz="10" samples="440" gpu="true">
-        <!-- <origin xyz="0.535 0 ${height_joint_velodyne}" rpy="0 0 0"/> -->
         <origin xyz="0.232 0 ${height_joint_velodyne}" rpy="0 0 0"/>
     </xacro:VLP-16>
@@ -278,11 +277,15 @@
             <visualize>true</visualize>
             <topic>data</topic>
-            <plugin filename="libgazebo_ros_imu_sensor.so" name="imu_plugin">
-                <topicName>imu/data</topicName>
+            <plugin filename="libgazebo_ros_imu_sensor.so" name="test">
+                <ros>
+                    <namespace>/sensing</namespace>
+                    <remapping>~/out:=imu/data</remapping>
+                </ros>
+                <topicName>imu/raw</topicName>
                 <bodyName>imu_link</bodyName>
                 <updateRateHZ>10.0</updateRateHZ>
                 <gaussianNoise>0.0</gaussianNoise>
                 <xyzOffset>0 0 0</xyzOffset>
-                <rpyOf7fset>0 0 0</rpyOf7fset>
+                <rpyOffset>0 0 0</rpyOffset>
                 <frameName>imu_link</frameName>
             </plugin>

Commit message: fix smagv.urdf.xacro

File: simulation/urdf/smagv/smagv.urdf.xacro (robot description, xacro)
@@ -10,6 +10,7 @@
     <xacro:property name="base_type"                value="0"/><!-- 0:base_link  1:base_footprint -->
     <xacro:property name="base_type_baselink"       value="0"/>
-    <xacro:property name="model_img_body"           value="$(find journal1-sim)/urdf/smagv/mesh/base/AGV0208_downsampling.${model_img_type}"/>
-    <!-- <xacro:property name="model_img_body"           value="$(find journal1-sim)/urdf/smagv/mesh/base/AGV0208.${model_img_type}"/> -->
+    <xacro:property name="model_img_body"           value="file://$(find journal1-sim)/urdf/smagv/mesh/base/AGV0208_downsampling_nocaster.${model_img_type}"/>
+    <xacro:property name="model_img_caster"           value="file://$(find journal1-sim)/urdf/smagv/mesh/base/caster.${model_img_type}"/>
+    <!-- <xacro:property name="model_img_body"           value="file://$(find journal1-sim)/urdf/smagv/mesh/base/AGV0208.${model_img_type}"/> -->
     <xacro:property name="base_height"              value="0"/>                                                                 <!-- -->
     <xacro:property name="base_height_gap"          value="${wh_radius}"/>                                                      <!-- -->
@@ -30,12 +31,12 @@
     <!-- ******************************************************************* -->
     <!-- <xacro:if value="${base_type == base_type_baselink}">                                                                          -->
-    <!--     <xacro:property name="model_img_body"   value="$(find journal1-sim)/urdf/smagv/mesh/base/AGV0208.${model_img_type}"/>       -->
+    <!--     <xacro:property name="model_img_body"   value="file://$(find journal1-sim)/urdf/smagv/mesh/base/AGV0208.${model_img_type}"/>       -->
     <!-- </xacro:if>                                                                                                                    -->
     <!-- <xacro:if value="${base_type != base_type_baselink}">                                                                          -->
-    <!--     <xacro:property name="model_img_body"   value="$(find journal1-sim)/urdf/smagv/mesh/footprint/AGV0208FT.${model_img_type}"/>-->
+    <!--     <xacro:property name="model_img_body"   value="file://$(find journal1-sim)/urdf/smagv/mesh/footprint/AGV0208FT.${model_img_type}"/>-->
     <!-- </xacro:if>                                                                                                                    -->
-    <xacro:property name="model_img_wheel_l"    value="$(find journal1-sim)/urdf/smagv/mesh/AGV_WHL_L.${model_img_type}"/>
-    <xacro:property name="model_img_wheel_r"    value="$(find journal1-sim)/urdf/smagv/mesh/AGV_WHL_R.${model_img_type}"/>
-    <xacro:property name="model_img_velodyne"   value="$(find journal1-sim)/urdf/smagv/mesh/VLP16.${model_img_type}"/>
+    <xacro:property name="model_img_wheel_l"    value="file://$(find journal1-sim)/urdf/smagv/mesh/AGV_WHL_L.${model_img_type}"/>
+    <xacro:property name="model_img_wheel_r"    value="file://$(find journal1-sim)/urdf/smagv/mesh/AGV_WHL_R.${model_img_type}"/>
+    <xacro:property name="model_img_velodyne"   value="file://$(find journal1-sim)/urdf/smagv/mesh/VLP16.${model_img_type}"/>
     <!-- ******************************************************************* -->
     <!-- spec , kansei moment                                                -->
@@ -248,7 +249,59 @@
         </joint>
     </xacro:if>
+    <xacro:macro name="caster" params="prefix parent xyz rpy model_img">
+        <!-- caster_support -->
+        <link name="${prefix}_caster_support">
+            <visual>
+                <geometry>
+                    <box size="0.01 0.01 0.01"/>
+                    <!-- <mesh filename="${model_img_caster}" /> -->
+                </geometry>
+                <!-- <origin xyz="0.44 0.15 0.21" rpy="0 0 0"/> -->
+                <origin xyz="0 0 0" rpy="0 0 0"/>
+                <material name="grey"/>
+            </visual>
+            <collision>
+                <geometry>
+                    <box size="0.01 0.01 0.01"/>
+                    <!-- <mesh filename="${model_img_caster}" /> -->
+                </geometry>
+                <!-- <origin xyz="0.44 0.15 0.21" rpy="0 0 0"/> -->
+                <origin xyz="0 0 0" rpy="0 0 0"/>
+            </collision>
+        </link>
+        <joint name="${prefix}_caster_support_joint" type="continuous">
+            <axis xyz="0 1 0"/>
+            <parent link="${parent}"/>
+            <child link="${prefix}_caster_support"/>
+            <origin xyz="${xyz}" rpy="${rpy}"/>
+        </joint>
+        <link name="${prefix}_caster_wheel">
+            <visual>
+            <geometry>
+                <!-- <cylinder length="0.005" radius="0.02"/> -->
+                <mesh filename="${model_img_caster}" />
+            </geometry>
+            <!-- <material name="black"/> -->
+            </visual>
+            <collision>
+            <geometry>
+                <!-- <cylinder length="0.005" radius="0.02"/> -->
+                <mesh filename="${model_img_caster}" />
+            </geometry>
+            </collision>
+        </link>
+        <joint name="${prefix}_caster_wheel_joint" type="fixed">
+            <!-- <axis xyz="0 1 0"/> -->
+            <parent link="${prefix}_caster_support"/>
+            <child link="${prefix}_caster_wheel"/>
+            <origin xyz="0 0 0" rpy="0 0 0"/>
+        </joint>
+    </xacro:macro>
     <!-- wheel -->
     <xacro:wheel_macro prefix="left_wheel"  parent="base_link" xyz="0 0.161 ${height_joint_wheel}"  rpy="${radians(-90)} 0 0" model_img="${model_img_wheel_l}"/>
     <xacro:wheel_macro prefix="right_wheel" parent="base_link" xyz="0 -0.161 ${height_joint_wheel}" rpy="${radians(-90)} 0 0" model_img="${model_img_wheel_r}"/>
+    <!-- caster -->
+    <xacro:caster prefix="right" parent="base_link" xyz="0.44 0.15 0.21" rpy="${radians(-90)} 0 0" model_img="${model_img_caster}"/>
+    <xacro:caster prefix="left" parent="base_link" xyz="0.44 -0.15 0.21" rpy="${radians(-90)} 0 0" model_img="${model_img_caster}"/>
     <!-- VLP-16 on Gazebo -->
     <xacro:include filename="$(find velodyne_description)/urdf/VLP-16.urdf.xacro"/>

Commit message: add caster

File: simulation/urdf/smagv/smagv.urdf.xacro (robot description, xacro)
@@ -11,5 +11,5 @@
     <xacro:property name="base_type_baselink"       value="0"/>
     <xacro:property name="model_img_body"           value="file://$(find journal1-sim)/urdf/smagv/mesh/base/AGV0208_downsampling_nocaster.${model_img_type}"/>
-    <xacro:property name="model_img_caster"           value="file://$(find journal1-sim)/urdf/smagv/mesh/base/caster.${model_img_type}"/>
+    <xacro:property name="model_img_caster"         value="file://$(find journal1-sim)/urdf/smagv/mesh/base/caster_origin_joint.${model_img_type}"/>
     <!-- <xacro:property name="model_img_body"           value="file://$(find journal1-sim)/urdf/smagv/mesh/base/AGV0208.${model_img_type}"/> -->
     <xacro:property name="base_height"              value="0"/>                                                                 <!-- -->
@@ -49,4 +49,11 @@
     <xacro:property name="wheel_iyy"  value="${wheel_ixx}"/>
     <xacro:property name="wheel_izz"  value="${(wheel_mass*(wh_length**2))/2.0}"/>
+    <!-- caster property -->
+    <xacro:property name="caster_radius"  value="0.074"/><!-- radius -->
+    <xacro:property name="caster_length"  value="0.03"/><!-- length -->
+    <xacro:property name="caster_mass" value="1.0"/>
+    <xacro:property name="caster_ixx" value="${(caster_mass*(3*(caster_radius**2)+(caster_length**2)))/12.0}"/>
+    <xacro:property name="caster_iyy" value="${caster_ixx}"/>
+    <xacro:property name="caster_izz" value="${(caster_mass*(caster_length**2))/2.0}"/>
     <!-- hight -->
     <!-- <xacro:if value="${base_type == base_type_baselink}">                  -->
@@ -252,10 +259,9 @@
         <!-- caster_support -->
         <link name="${prefix}_caster_support">
-            <visual>
+            <visual name="${prefix}_visual">
                 <geometry>
                     <box size="0.01 0.01 0.01"/>
                     <!-- <mesh filename="${model_img_caster}" /> -->
                 </geometry>
-                <!-- <origin xyz="0.44 0.15 0.21" rpy="0 0 0"/> -->
                 <origin xyz="0 0 0" rpy="0 0 0"/>
                 <material name="grey"/>
@@ -266,7 +272,11 @@
                     <!-- <mesh filename="${model_img_caster}" /> -->
                 </geometry>
-                <!-- <origin xyz="0.44 0.15 0.21" rpy="0 0 0"/> -->
                 <origin xyz="0 0 0" rpy="0 0 0"/>
             </collision>
+            <inertial>
+                <origin xyz="0 0 0" rpy="0 0 0"/>
+                <mass value="0.5"/>
+                <inertia ixx="0.01" ixy="0" ixz="0" iyy="0.01" iyz="0" izz="0.01"/>
+            </inertial>
         </link>
         <joint name="${prefix}_caster_support_joint" type="continuous">
@@ -278,23 +288,37 @@
         <link name="${prefix}_caster_wheel">
             <visual>
-            <geometry>
-                <!-- <cylinder length="0.005" radius="0.02"/> -->
-                <mesh filename="${model_img_caster}" />
-            </geometry>
-            <!-- <material name="black"/> -->
+                <geometry>
+                    <cylinder length="${caster_length}" radius="${caster_radius}"/>
+                    <!-- <mesh filename="${model_img_caster}" /> -->
+                </geometry>
+                <origin xyz="0 0 0" rpy="0 0 0"/>
+                <material name="black"/>
             </visual>
             <collision>
-            <geometry>
-                <!-- <cylinder length="0.005" radius="0.02"/> -->
-                <mesh filename="${model_img_caster}" />
-            </geometry>
+                <geometry>
+                    <cylinder length="${caster_length}" radius="${caster_radius}"/>
+                    <!-- <mesh filename="${model_img_caster}" /> -->
+                </geometry>
+                <origin xyz="0 0 0" rpy="0 0 0"/>
             </collision>
-        </link>
-        <joint name="${prefix}_caster_wheel_joint" type="fixed">
-            <!-- <axis xyz="0 1 0"/> -->
+            <inertial>
+                <origin xyz="0 0 0" rpy="0 0 0"/>
+                <mass value="${caster_mass}"/>
+                <inertia ixx="${caster_ixx}" ixy="0" ixz="0" iyy="${caster_iyy}" iyz="0" izz="${caster_izz}"/>
+            </inertial>
+        </link>
+        <joint name="${prefix}_caster_wheel_joint" type="continuous">
+            <axis xyz="0 0 1"/>
             <parent link="${prefix}_caster_support"/>
             <child link="${prefix}_caster_wheel"/>
-            <origin xyz="0 0 0" rpy="0 0 0"/>
-        </joint>
+            <origin xyz="0.04 0.136 0" rpy="0 0 0"/>
+        </joint>
+        <gazebo reference="${prefix}_caster_wheel">
+            <mu1 value="1.0" />
+            <mu2 value="1.0" />
+            <kp  value="10000000.0" />
+            <kd  value="1.0" />
+            <material name="white"/>
+        </gazebo>
     </xacro:macro>
     <!-- wheel -->

Commit message: fix launch

File: simulation/urdf/smagv/smagv.urdf.xacro (robot description, xacro)
@@ -11,4 +11,5 @@
     <xacro:property name="base_type_baselink"       value="0"/>
     <xacro:property name="model_img_body"           value="file://$(find journal1-sim)/urdf/smagv/mesh/base/AGV0208_downsampling_nocaster.${model_img_type}"/>
+    <!-- <xacro:property name="model_img_body"           value="file://$(find journal1-sim)/urdf/smagv/mesh/base/AGV0208_downsampling.${model_img_type}"/> -->
     <xacro:property name="model_img_caster"         value="file://$(find journal1-sim)/urdf/smagv/mesh/base/caster_origin_joint.${model_img_type}"/>
     <!-- <xacro:property name="model_img_body"           value="file://$(find journal1-sim)/urdf/smagv/mesh/base/AGV0208.${model_img_type}"/> -->
@@ -203,4 +204,5 @@
     <gazebo>
         <plugin filename="libgazebo_ros2_control.so" name="gazebo_ros2_control">
+            <!-- <robot_namespace>robot1</robot_namespace> -->
             <robot_param>robot_description</robot_param>
             <robot_param_node>robot_state_publisher</robot_param_node>
@@ -330,5 +332,6 @@
     <!-- VLP-16 on Gazebo -->
     <xacro:include filename="$(find velodyne_description)/urdf/VLP-16.urdf.xacro"/>
-    <xacro:VLP-16 parent="base_link" name="velodyne" topic="/sensing/lidar/concatenated/pointcloud" hz="10" samples="440" gpu="true">
+    <!-- <xacro:VLP-16 parent="base_link" name="velodyne_top" topic="/sensing/lidar/top/pointcloud_raw_ex" hz="10" samples="440" gpu="true" organize_cloud="true"> -->
+    <xacro:VLP-16 parent="base_link" name="velodyne_top" topic="/robot1/sensing/lidar/top/pointcloud_raw_ex" hz="10" samples="440" gpu="true" organize_cloud="true">
         <origin xyz="0.232 0 ${height_joint_velodyne}" rpy="0 0 0"/>
     </xacro:VLP-16>
